Commit message: actualizacion

File: src/rosbot/urdf/include.xacro (robot description, xacro)
@@ -22,5 +22,5 @@
     </material>
     <!-- Especificar colores de gazebo -->
-    <gazebo reference="base_link">
+    <gazebo reference="chasis">
         <material>Gazebo/Blue</material>
     </gazebo>

File: src/rosbot/urdf/rosbot.urdf (robot description, URDF)
Before this commit: robot rosbot, 9 links, 8 joints
Links:
- removed link base_link
- added link chasis, mass 30; collision mesh filename=package://rosbot/meshes/box.STL scale=0.001 0.001 0.001; visual mesh filename=package://rosbot/meshes/box.STL scale=0.001 0.001 0.001
- added link lidar_link, mass 0.125; collision cylinder length=0.05 radius=0.05; visual cylinder length=0.09 radius=0.05
Joints:
- added joint lidar_joint: type fixed, parent chasis, child lidar_link, origin xyz= 0.2 0 0.15 rpy=0 0 0
- joint base_camara: parent base_link -> chasis
- joint base_joint: child base_link -> chasis
- joint joint_left_rear_wheel: parent base_link -> chasis
- joint joint_left_wheel_front: parent base_link -> chasis
- joint joint_right_rear_wheel: parent base_link -> chasis
- joint joint_right_wheel_front: parent base_link -> chasis

File: src/rosbot/urdf/rosbot.urdf.xacro (robot description, xacro)
@@ -22,5 +22,5 @@
       específicos del robot dentro del entorno de simulación. Cada etiqueta
       `<gazebo reference="..." >` se refiere a un componente en particular, como
-      `base_link` o las diferentes ruedas, y asigna un material específico para
+      `chasis` o las diferentes ruedas, y asigna un material específico para
       su visualización en Gazebo.
     @note Es necesario modificar la ruta del archivo "include.xacro" según la
@@ -34,9 +34,9 @@
   <joint name="base_joint" type="fixed">
     <parent link="base_footprint"/>
-    <child link="base_link"/>
+    <child link="chasis"/>
     <origin xyz="0 0 0.19" />
   </joint>
   <!--Chasis-->
-  <link name="base_link">
+  <link name="chasis">
     <visual>
       <geometry>
@@ -70,5 +70,5 @@
   </link>
   <joint name="base_camara" type="fixed">
-    <parent link="base_link"/>
+    <parent link="chasis"/>
     <child link="camara_link"/>
     <origin xyz=" 0.30 0 0.1" rpy="0 -0.156 0"/>
@@ -97,5 +97,5 @@
   </link>
   <joint name="lidar_joint" type="fixed">
-    <parent link="base_link"/>
+    <parent link="chasis"/>
     <child link="lidar_link"/>
     <origin xyz=" 0.2 0 0.15" rpy="0 0 0"/>
@@ -160,5 +160,5 @@
   </link>
   <joint name="joint_right_wheel" type="continuous">
-    <parent link="base_link"/>
+    <parent link="chasis"/>
     <child link="right_wheel"/>
     <origin xyz="-0.27 -0.295 -0.07" rpy="1.57 0 0"/>
@@ -185,5 +185,5 @@
   </link>
   <joint name="joint_left_wheel" type="continuous">
-    <parent link="base_link"/>
+    <parent link="chasis"/>
     <child link="left_wheel"/>
     <origin xyz="-0.27 0.295 -0.07" rpy="1.57 0 0"/>
@@ -193,5 +193,5 @@
   </link>
   <joint name="master_joint" type="revolute">
-    <parent link="base_link"/>
+    <parent link="chasis"/>
     <child link="master"/>
     <origin xyz="0 0 0" rpy= "1.57 0 0"/>
@@ -230,5 +230,5 @@
   </link>
   <joint name="joint_right_wheel_front" type="revolute">
-    <parent link="base_link"/>
+    <parent link="chasis"/>
     <child link="right_wheel_front_assembly"/>
     <origin xyz="0.27 -0.295 -0.07" rpy="1.57 0 0"/>
@@ -275,5 +275,5 @@
   </link>
   <joint name="joint_left_wheel_front" type="revolute">
-    <parent link="base_link"/>
+    <parent link="chasis"/>
     <child link="left_wheel_front_assembly"/>
     <origin xyz="0.27 0.295 -0.07" rpy="1.57 0 0"/>

Commit message: actualizacion 4

File: src/rosbot/urdf/include.xacro (robot description, xacro)
@@ -20,4 +20,7 @@
     <material name="blue">
         <color rgba="0.2 0.2 1 1"/>
+    </material>
+    <material name="grey">
+        <color rgba="0 0 0 1"/>
     </material>
     <!-- Especificar colores de gazebo -->

File: src/rosbot/urdf/rosbot.urdf.xacro (robot description, xacro)
@@ -56,6 +56,155 @@
     </xacro:inertial_chasis>
   </link>
+  <!--Right-->
+  <link name="right_wheel">
+    <visual>
+      <geometry>
+         <cylinder length="0.08" radius="0.12"/>
+      </geometry>
+      <origin xyz="0 0 0"/>
+      <material name="white"/>
+    </visual>
+    <collision>
+      <origin xyz="0 0 0"/>
+      <geometry>
+        <cylinder length="0.08" radius="0.12"/>
+      </geometry>
+    </collision>
+    <xacro:inertial_wheel mass="1.0" length="0.08" radius="0.12">
+      <origin xyz="0 0 0" rpy="0 0 0"/>
+    </xacro:inertial_wheel>
+  </link>
+  <joint name="joint_right_wheel" type="continuous">
+    <parent link="chasis"/>
+    <child link="right_wheel"/>
+    <origin xyz="-0.27 -0.295 -0.07" rpy="1.57 0 0"/>
+    <axis xyz="0 0 1"/>
+  </joint>
+ <!--Left -->
+  <link name="left_wheel">
+    <visual>
+      <geometry>
+         <cylinder length="0.08" radius="0.12"/>
+      </geometry>
+      <origin xyz="0 0 0"/>
+      <material name="white"/>
+    </visual>
+    <collision>
+      <origin xyz="0 0 0"/>
+      <geometry>
+        <cylinder length="0.08" radius="0.12"/>
+      </geometry>
+    </collision>
+    <xacro:inertial_wheel mass="1.0" length="0.08" radius="0.12">
+      <origin xyz="0 0 0" rpy="0 0 0"/>
+    </xacro:inertial_wheel>
+  </link>
+  <joint name="joint_left_wheel" type="continuous">
+    <parent link="chasis"/>
+    <child link="left_wheel"/>
+    <origin xyz="-0.27 0.295 -0.07" rpy="1.57 0 0"/>
+    <axis xyz="0 0 1"/>
+  </joint>
+  <link name="master">
+  </link>
+  <joint name="master_joint" type="revolute">
+    <parent link="chasis"/>
+    <child link="master"/>
+    <origin xyz="0 0 0" rpy= "1.57 0 0"/>
+    <axis xyz="0 1 0"/>
+    <limit effort="100" velocity="1" lower="-0.78" upper="0.78"/>
+  </joint>
+  <link name="right_wheel_front_assembly">
+    <visual>
+      <geometry>
+         <cylinder length="0.001" radius="0.04"/>
+      </geometry>
+      <origin xyz="0 0 0"/>
+      <material name="white"/>
+    </visual>
+    <xacro:inertial_wheel mass="1.0" length="0.001" radius="0.04">
+      <origin xyz="0 0 0" rpy="0 0 0"/>
+    </xacro:inertial_wheel>
+  </link>
+  <link name="right_wheel_front">
+    <visual>
+      <geometry>
+         <cylinder length="0.08" radius="0.12"/>
+      </geometry>
+      <origin xyz="0 0 0"/>
+      <material name="white"/>
+    </visual>
+    <collision>
+      <origin xyz="0 0 0"/>
+      <geometry>
+        <cylinder length="0.08" radius="0.12"/>
+      </geometry>
+    </collision>
+    <xacro:inertial_wheel mass="1.0" length="0.08" radius="0.12">
+      <origin xyz="0 0 0" rpy="0 0 0"/>
+    </xacro:inertial_wheel>
+  </link>
+  <joint name="joint_right_wheel_front" type="revolute">
+    <parent link="chasis"/>
+    <child link="right_wheel_front_assembly"/>
+    <origin xyz="0.27 -0.295 -0.07" rpy="1.57 0 0"/>
+    <axis xyz="0 1 0"/>
+    <limit effort="100" velocity="1" lower="-0.78" upper="0.78"/>
+    <mimic joint="master_joint" multiplier="1.0" offset="0"/>
+  </joint>
+  <joint name="right_wheel_joint" type="continuous">
+    <parent link="right_wheel_front_assembly"/>
+    <child link="right_wheel_front"/>
+    <origin xyz="0.0 0 0" rpy="0 0 0"/>
+    <axis xyz="0 0 1"/>
+    <limit effort="100" velocity="1"/>
+  </joint>
+  <link name="left_wheel_front_assembly">
+      <visual>
+      <geometry>
+         <cylinder length="0.001" radius="0.04"/>
+      </geometry>
+      <origin xyz="0 0 0"/>
+      <material name="white"/>
+    </visual>
+    <xacro:inertial_wheel mass="1.0" length="0.001" radius="0.04">
+      <origin xyz="0 0 0" rpy="0 0 0"/>
+    </xacro:inertial_wheel>
+  </link>
+  <link name="left_wheel_front">
+    <visual>
+      <geometry>
+         <cylinder length="0.08" radius="0.12"/>
+      </geometry>
+      <origin xyz="0 0 0"/>
+      <material name="white"/>
+    </visual>
+    <collision>
+      <origin xyz="0 0 0"/>
+      <geometry>
+        <cylinder length="0.08" radius="0.12"/>
+      </geometry>
+    </collision>
+    <xacro:inertial_wheel mass="1.0" length="0.08" radius="0.12">
+      <origin xyz="0 0 0" rpy="0 0 0"/>
+    </xacro:inertial_wheel>
+  </link>
+  <joint name="joint_left_wheel_front" type="revolute">
+    <parent link="chasis"/>
+    <child link="left_wheel_front_assembly"/>
+    <origin xyz="0.27 0.295 -0.07" rpy="1.57 0 0"/>
+    <axis xyz="0 1 0"/>
+    <limit effort="100" velocity="1" lower="-0.78" upper="0.78"/>
+    <mimic joint="master_joint" multiplier="1.0" offset="0"/>
+  </joint>
+    <joint name="left_wheel_joint" type="continuous">
+    <parent link="left_wheel_front_assembly"/>
+    <child link="left_wheel_front"/>
+    <origin xyz="0.0 0 0" rpy="0 0 0"/>
+    <axis xyz="0 0 1"/>
+    <limit effort="100" velocity="1"/>
+  </joint>
   <!--camara-->
-  <link name= "camara_link">
+  <link name="camera_link">
     <visual>
       <origin xyz="0 0 0" rpy="0 -0.156 0"/>
@@ -63,17 +212,62 @@
         <box size="0.04 0.17 0.03"/>
       </geometry>
-      <material name="orange"/>
-    </visual>
-    <xacro:inertial_chasis mass="0.181" x="0.05" y="0.05" z="0.05">
+    </visual>
+    <collision>
+      <origin xyz="0 0 0" rpy="0 -0.156 0"/>
+      <geometry>
+        <box size="0.04 0.17 0.03"/>
+      </geometry>
+    </collision>
+    <xacro:inertial_chasis mass="0.181" x="0.04" y="0.17" z="0.03">
       <origin xyz="0 0 0" rpy="0 0 0"/>
     </xacro:inertial_chasis>
   </link>
-  <joint name="base_camara" type="fixed">
-    <parent link="chasis"/>
-    <child link="camara_link"/>
+  <joint name="camera_joint" type="fixed">
+    <parent link="chasis"/>
+    <child link="camera_link"/>
     <origin xyz=" 0.30 0 0.1" rpy="0 -0.156 0"/>
-    <limit effort="100" velocity="1" lower="-0.78" upper="0.78"/>
-    <axis xyz="0 1 0"/>
-  </joint>
+  </joint>
+  <link name="camera_depth_frame"/>
+  <joint name="camera_depth_joint" type="fixed">
+    <origin xyz="0 0 0" rpy="0 0 0"/>
+    <parent link="camera_link"/>
+    <child link="camera_depth_frame"/>
+  </joint>
+  <gazebo reference="camera_link">
+    <sensor name="depth_camera" type="depth">
+      <visualize>true</visualize>
+      <update_rate>30.0</update_rate>
+      <camera name="camera">
+        <horizontal_fov>1.047198</horizontal_fov>
+        <image>
+          <width>640</width>
+          <height>480</height>
+          <format>R8G8B8</format>
+        </image>
+        <clip>
+          <near>0.05</near>
+          <far>3</far>
+        </clip>
+      </camera>
+      <plugin name="depth_camera_controller" filename="libgazebo_ros_camera.so">
+        <baseline>0.2</baseline>
+        <alwaysOn>true</alwaysOn>
+        <updateRate>0.0</updateRate>
+        <frameName>camera_depth_frame</frameName>
+        <pointCloudCutoff>0.5</pointCloudCutoff>
+        <pointCloudCutoffMax>3.0</pointCloudCutoffMax>
+        <distortionK1>0</distortionK1>
+        <distortionK2>0</distortionK2>
+        <distortionK3>0</distortionK3>
+        <distortionT1>0</distortionT1>
+        <distortionT2>0</distortionT2>
+        <CxPrime>0</CxPrime>
+        <Cx>0</Cx>
+        <Cy>0</Cy>
+        <focalLength>0</focalLength>
+        <hackBaseline>0</hackBaseline>
+      </plugin>
+    </sensor>
+  </gazebo>
   <!--lidar-->
    <link name="lidar_link">
@@ -140,152 +334,89 @@
     <material>Gazebo/Black</material>
   </gazebo>
-  <!--Right-->
-  <link name="right_wheel">
-    <visual>
-      <geometry>
-         <cylinder length="0.08" radius="0.12"/>
-      </geometry>
-      <origin xyz="0 0 0"/>
-      <material name="white"/>
-    </visual>
-    <collision>
-      <origin xyz="0 0 0"/>
-      <geometry>
-        <cylinder length="0.08" radius="0.12"/>
-      </geometry>
-    </collision>
-    <xacro:inertial_wheel mass="1.0" length="0.08" radius="0.12">
-      <origin xyz="0 0 0" rpy="0 0 0"/>
-    </xacro:inertial_wheel>
-  </link>
-  <joint name="joint_right_wheel" type="continuous">
-    <parent link="chasis"/>
-    <child link="right_wheel"/>
-    <origin xyz="-0.27 -0.295 -0.07" rpy="1.57 0 0"/>
-    <axis xyz="0 0 1"/>
-  </joint>
- <!--Left -->
-  <link name="left_wheel">
-    <visual>
-      <geometry>
-         <cylinder length="0.08" radius="0.12"/>
-      </geometry>
-      <origin xyz="0 0 0"/>
-      <material name="white"/>
-    </visual>
-    <collision>
-      <origin xyz="0 0 0"/>
-      <geometry>
-        <cylinder length="0.08" radius="0.12"/>
-      </geometry>
-    </collision>
-    <xacro:inertial_wheel mass="1.0" length="0.08" radius="0.12">
-      <origin xyz="0 0 0" rpy="0 0 0"/>
-    </xacro:inertial_wheel>
-  </link>
-  <joint name="joint_left_wheel" type="continuous">
-    <parent link="chasis"/>
-    <child link="left_wheel"/>
-    <origin xyz="-0.27 0.295 -0.07" rpy="1.57 0 0"/>
-    <axis xyz="0 0 1"/>
-  </joint>
-  <link name="master">
-  </link>
-  <joint name="master_joint" type="revolute">
-    <parent link="chasis"/>
-    <child link="master"/>
-    <origin xyz="0 0 0" rpy= "1.57 0 0"/>
-    <axis xyz="0 1 0"/>
-    <limit effort="100" velocity="1" lower="-0.78" upper="0.78"/>
-  </joint>
-  <link name="right_wheel_front_assembly">
-    <visual>
-      <geometry>
-         <cylinder length="0.001" radius="0.04"/>
-      </geometry>
-      <origin xyz="0 0 0"/>
-      <material name="white"/>
-    </visual>
-    <xacro:inertial_wheel mass="1.0" length="0.001" radius="0.04">
-      <origin xyz="0 0 0" rpy="0 0 0"/>
-    </xacro:inertial_wheel>
-  </link>
-  <link name="right_wheel_front">
-    <visual>
-      <geometry>
-         <cylinder length="0.08" radius="0.12"/>
-      </geometry>
-      <origin xyz="0 0 0"/>
-      <material name="white"/>
-    </visual>
-    <collision>
-      <origin xyz="0 0 0"/>
-      <geometry>
-        <cylinder length="0.08" radius="0.12"/>
-      </geometry>
-    </collision>
-    <xacro:inertial_wheel mass="1.0" length="0.08" radius="0.12">
-      <origin xyz="0 0 0" rpy="0 0 0"/>
-    </xacro:inertial_wheel>
-  </link>
-  <joint name="joint_right_wheel_front" type="revolute">
-    <parent link="chasis"/>
-    <child link="right_wheel_front_assembly"/>
-    <origin xyz="0.27 -0.295 -0.07" rpy="1.57 0 0"/>
-    <axis xyz="0 1 0"/>
-    <limit effort="100" velocity="1" lower="-0.78" upper="0.78"/>
-    <!--<mimic joint="master_joint" multiplier="1.0" offset="0"/>-->
-  </joint>
-  <joint name="right_wheel_joint" type="continuous">
-    <parent link="right_wheel_front_assembly"/>
-    <child link="right_wheel_front"/>
-    <origin xyz="0.0 0 0" rpy="0 0 0"/>
-    <axis xyz="0 0 1"/>
-    <limit effort="100" velocity="1"/>
-  </joint>
-  <link name="left_wheel_front_assembly">
-      <visual>
-      <geometry>
-         <cylinder length="0.001" radius="0.04"/>
-      </geometry>
-      <origin xyz="0 0 0"/>
-      <material name="white"/>
-    </visual>
-    <xacro:inertial_wheel mass="1.0" length="0.001" radius="0.04">
-      <origin xyz="0 0 0" rpy="0 0 0"/>
-    </xacro:inertial_wheel>
-  </link>
-  <link name="left_wheel_front">
-    <visual>
-      <geometry>
-         <cylinder length="0.08" radius="0.12"/>
-      </geometry>
-      <origin xyz="0 0 0"/>
-      <material name="white"/>
-    </visual>
-    <collision>
-      <origin xyz="0 0 0"/>
-      <geometry>
-        <cylinder length="0.08" radius="0.12"/>
-      </geometry>
-    </collision>
-    <xacro:inertial_wheel mass="1.0" length="0.08" radius="0.12">
-      <origin xyz="0 0 0" rpy="0 0 0"/>
-    </xacro:inertial_wheel>
-  </link>
-  <joint name="joint_left_wheel_front" type="revolute">
-    <parent link="chasis"/>
-    <child link="left_wheel_front_assembly"/>
-    <origin xyz="0.27 0.295 -0.07" rpy="1.57 0 0"/>
-    <axis xyz="0 1 0"/>
-    <limit effort="100" velocity="1" lower="-0.78" upper="0.78"/>
-    <!--<mimic joint="master_joint" multiplier="1.0" offset="0"/>-->
-  </joint>
-    <joint name="left_wheel_joint" type="continuous">
-    <parent link="left_wheel_front_assembly"/>
-    <child link="left_wheel_front"/>
-    <origin xyz="0.0 0 0" rpy="0 0 0"/>
-    <axis xyz="0 0 1"/>
-    <limit effort="100" velocity="1"/>
-  </joint>
+  <!-- IMU -->
+  <link name="imu_link">
+    <inertial>
+      <origin xyz="0 0 0" rpy="0 0 0"/>
+      <mass value="0.01"/>
+      <inertia ixx="0.001" ixy="0" ixz="0" iyy="0.001" iyz="0" izz="0.001"/>
+    </inertial>
+    <visual>
+      <geometry>
+        <box size="0.03 0.03 0.01"/>
+      </geometry>
+      <origin xyz="0 0 0" rpy="0 0 0"/>
+      <material name="grey"/>
+    </visual>
+  </link>
+  <joint name="imu_joint" type="fixed">
+    <parent link="chasis"/>
+    <child link="imu_link"/>
+    <origin xyz="0.0 0.0 0.0" rpy="0 0 0"/>
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