Commit message: actualizacion 5

File: src/rosbot/urdf/include.xacro (robot description, xacro)
@@ -1,14 +1,4 @@
 <?xml version="1.0"?>
 <robot xmlns:xacro="http://www.ros.org/wiki/xacro" >
-    <!--
-    Descripción:
-    Este archivo Xacro define configuraciones estándar de materiales y macros para calcular las inercias de componentes específicos de un modelo de robot.
-    Se utiliza en conjunto con un archivo URDF para asignar colores a las diferentes partes del robot y para realizar cálculos automáticos de inercias basados en las dimensiones y masas de los componentes.
-    - Materiales: Se definen tres colores (blanco, naranja y azul) que pueden ser aplicados a las partes visuales del robot.
-    - Cálculo de inercias: Se proporcionan macros para calcular la matriz de inercia de componentes como el chasis y las ruedas del robot.
-    Detalles:
-    - La macro `inertial_chasis` calcula la inercia de un chasis rectangular utilizando sus dimensiones y masa.
-    - La macro `inertial_wheel` calcula la inercia de una rueda cilíndrica basándose en su masa, longitud y radio.
-    -->
     <!-- Especificación de colores -->
     <material name="white">
@@ -30,18 +20,24 @@
     <gazebo reference="right_wheel">
         <material>Gazebo/White</material>
+        <mu1>0.2</mu1>
+        <mu2>0.2</mu2>
     </gazebo>
     <gazebo reference="left_wheel">
         <material>Gazebo/White</material>
+        <mu1>0.2</mu1>
+        <mu2>0.2</mu2>
     </gazebo>
     <gazebo reference="right_wheel_front">
         <material>Gazebo/White</material>
+        <mu1>0.2</mu1>
+        <mu2>0.2</mu2>
     </gazebo>
     <gazebo reference="left_wheel_front">
         <material>Gazebo/White</material>
+        <mu1>0.2</mu1>
+        <mu2>0.2</mu2>
     </gazebo>
-    <!-- Especificación de cálculos estándar de inercias: https://en.wikipedia.org/wiki/List_of_moments_of_inertia -->
-    <!-- Estas macros utilizan la funcionalidad matemática de Xacro -->
     <!-- Macro para calcular la inercia de un chasis rectangular -->
-    <xacro:macro name="inertial_chasis" params="mass x y z *origin">
+    <xacro:macro name="inertial_box" params="mass x y z *origin">
         <inertial>
             <xacro:insert_block name="origin"/>
@@ -53,5 +49,5 @@
     </xacro:macro>
     <!-- Macro para calcular la inercia de una rueda cilíndrica -->
-    <xacro:macro name="inertial_wheel" params="mass length radius *origin">
+    <xacro:macro name="inertial_cylinder" params="mass length radius *origin">
         <inertial>
             <xacro:insert_block name="origin"/>

File: src/rosbot/urdf/rosbot.urdf (robot description, URDF)
Before this commit: robot rosbot, 10 links, 9 joints
Links:
- removed link camara_link
- added link camera_depth_frame
- added link camera_link; collision box size=0.04 0.17 0.03; visual box size=0.04 0.17 0.03
- added link master
- link left_rear_wheel: mass 1 -> None
- link left_wheel_front: mass 1 -> None
- link left_wheel_front_assembly: mass 0.01 -> None
- link lidar_link: geometry collision cylinder length=0.05 radius=0.05; visual cylinder length=0.05 radius=0.05
- link right_rear_wheel: mass 1 -> None
- link right_wheel_front: mass 1 -> None
- link right_wheel_front_assembly: mass 0.01 -> None
Joints:
- removed joint base_camara
- added joint camera_depth_joint: type fixed, parent camera_link, child camera_depth_frame, origin xyz=0 0 0 rpy=0 0 0
- added joint camera_joint: type fixed, parent chasis, child camera_link, origin xyz= 0.30 0 0.1 rpy=0 -0.156 0
- added joint master_joint: type revolute, parent chasis, child master, origin xyz=0 0 0 rpy=1.57 0 0, axis 0 1 0, limit lower=-0.78 upper=0.78 effort=100 velocity=1
- joint joint_left_wheel_front: mimic (none) -> joint=master_joint multiplier=1.0 offset=0
- joint joint_right_wheel_front: mimic (none) -> joint=master_joint multiplier=1.0 offset=0

File: src/rosbot/urdf/rosbot.urdf.xacro (robot description, xacro)
@@ -1,32 +1,3 @@
 <?xml version="1.0"?>
-<!--
-    @file rosbot.urdf.xacro
-    @brief Descripción del robot móvil Rosbot utilizando Xacro y URDF.
-    Este archivo define la estructura, visualización y propiedades físicas del
-    robot móvil Rosbot. Utiliza macros Xacro para incluir elementos comunes y
-    define las características de los componentes principales del robot, tales
-    como el chasis y las ruedas. Además, configura los materiales y la simulación
-    en Gazebo para la visualización y simulación del robot en un entorno 3D.
-    Características principales:
-    - Incluye un archivo "include.xacro" que contiene definiciones comunes como
-      colores y cálculos de inercias.
-    - Define los enlaces (links) para el chasis, las ruedas y otras partes del robot.
-    - Configura las uniones (joints) entre los diferentes componentes del robot,
-      incluyendo las restricciones y la dinámica de las ruedas.
-    - Aplica materiales específicos para la visualización en Gazebo, los cuales
-      están definidos en un archivo separado.
-    - Las inercias de los componentes, tales como el chasis y las ruedas, son
-      calculadas automáticamente mediante macros definidas en un archivo separado.
-    - En la sección que define los parámetros para la simulación en Gazebo, se
-      utilizan etiquetas `<gazebo>` para personalizar la apariencia de componentes
-      específicos del robot dentro del entorno de simulación. Cada etiqueta
-      `<gazebo reference="..." >` se refiere a un componente en particular, como
-      `chasis` o las diferentes ruedas, y asigna un material específico para
-      su visualización en Gazebo.
-    @note Es necesario modificar la ruta del archivo "include.xacro" según la
-    estructura de directorios de tu proyecto.
-    @usage Este archivo es utilizado en la simulación del robot Rosbot en entornos
-    como RViz y Gazebo, y puede ser integrado en lanzadores ROS2 para su ejecución.
--->
 <robot xmlns:xacro="http://www.ros.org/wiki/xacro" name="rosbot">
   <xacro:include filename="include.xacro" />
@@ -52,7 +23,9 @@
       </geometry>
     </collision>
-    <xacro:inertial_chasis mass="20" x="0.762" y="0.35" z="0.15">
-      <origin xyz="0 0 0" rpy="0 0 0"/>
-    </xacro:inertial_chasis>
+    <inertial>
+      <origin xyz="-0.381 0.2 -0.075" rpy = "1.57 0 0"/>
+      <mass value="30"/>
+      <inertia  ixx="456250.0" ixy="0" ixz="0" iyy="1844000.0" iyz="0" izz="1500250.0" />
+    </inertial>
   </link>
   <!--Right-->
@@ -71,9 +44,9 @@
       </geometry>
     </collision>
-    <xacro:inertial_wheel mass="1.0" length="0.08" radius="0.12">
-      <origin xyz="0 0 0" rpy="0 0 0"/>
-    </xacro:inertial_wheel>
-  </link>
-  <joint name="joint_right_wheel" type="continuous">
+    <xacro:inertial_cylinder mass="1.0" length="0.08" radius="0.12">
+      <origin xyz="0 0 0" rpy="0 0 0"/>
+    </xacro:inertial_cylinder>
+  </link>
+  <joint name="joint_right_rear_wheel" type="continuous">
     <parent link="chasis"/>
     <child link="right_wheel"/>
@@ -96,9 +69,9 @@
       </geometry>
     </collision>
-    <xacro:inertial_wheel mass="1.0" length="0.08" radius="0.12">
-      <origin xyz="0 0 0" rpy="0 0 0"/>
-    </xacro:inertial_wheel>
-  </link>
-  <joint name="joint_left_wheel" type="continuous">
+    <xacro:inertial_cylinder mass="1.0" length="0.08" radius="0.12">
+      <origin xyz="0 0 0" rpy="0 0 0"/>
+    </xacro:inertial_cylinder>
+  </link>
+  <joint name="joint_left_rear_wheel" type="continuous">
     <parent link="chasis"/>
     <child link="left_wheel"/>
@@ -123,7 +96,7 @@
       <material name="white"/>
     </visual>
-    <xacro:inertial_wheel mass="1.0" length="0.001" radius="0.04">
-      <origin xyz="0 0 0" rpy="0 0 0"/>
-    </xacro:inertial_wheel>
+    <xacro:inertial_cylinder mass="1.0" length="0.001" radius="0.04">
+      <origin xyz="0 0 0" rpy="0 0 0"/>
+    </xacro:inertial_cylinder>
   </link>
   <link name="right_wheel_front">
@@ -141,7 +114,7 @@
       </geometry>
     </collision>
-    <xacro:inertial_wheel mass="1.0" length="0.08" radius="0.12">
-      <origin xyz="0 0 0" rpy="0 0 0"/>
-    </xacro:inertial_wheel>
+    <xacro:inertial_cylinder mass="1.0" length="0.08" radius="0.12">
+      <origin xyz="0 0 0" rpy="0 0 0"/>
+    </xacro:inertial_cylinder>
   </link>
   <joint name="joint_right_wheel_front" type="revolute">
@@ -168,7 +141,7 @@
       <material name="white"/>
     </visual>
-    <xacro:inertial_wheel mass="1.0" length="0.001" radius="0.04">
-      <origin xyz="0 0 0" rpy="0 0 0"/>
-    </xacro:inertial_wheel>
+    <xacro:inertial_cylinder mass="1.0" length="0.001" radius="0.04">
+      <origin xyz="0 0 0" rpy="0 0 0"/>
+    </xacro:inertial_cylinder>
   </link>
   <link name="left_wheel_front">
@@ -186,7 +159,7 @@
       </geometry>
     </collision>
-    <xacro:inertial_wheel mass="1.0" length="0.08" radius="0.12">
-      <origin xyz="0 0 0" rpy="0 0 0"/>
-    </xacro:inertial_wheel>
+    <xacro:inertial_cylinder mass="1.0" length="0.08" radius="0.12">
+      <origin xyz="0 0 0" rpy="0 0 0"/>
+    </xacro:inertial_cylinder>
   </link>
   <joint name="joint_left_wheel_front" type="revolute">
@@ -219,7 +192,7 @@
       </geometry>
     </collision>
-    <xacro:inertial_chasis mass="0.181" x="0.04" y="0.17" z="0.03">
-      <origin xyz="0 0 0" rpy="0 0 0"/>
-    </xacro:inertial_chasis>
+    <xacro:inertial_box mass="0.181" x="0.04" y="0.17" z="0.03">
+      <origin xyz="0 0 0" rpy="0 0 0"/>
+    </xacro:inertial_box>
   </link>
   <joint name="camera_joint" type="fixed">
@@ -337,5 +310,4 @@
   <link name="imu_link">
     <inertial>
-      <origin xyz="0 0 0" rpy="0 0 0"/>
       <mass value="0.01"/>
       <inertia ixx="0.001" ixy="0" ixz="0" iyy="0.001" iyz="0" izz="0.001"/>
@@ -374,12 +346,4 @@
         </orientation>
       </imu>
-      <plugin name="imu_plugin" filename="libgazebo_ros_imu.so">
-        <ros>
-          <namespace>/rosbot</namespace>
-          <remapping>~/imu/data:=/imu/data</remapping>
-        </ros>
-        <update_rate>50.0</update_rate>
-        <alwaysOn>true</alwaysOn>
-      </plugin>
     </sensor>
   </gazebo>
@@ -402,5 +366,5 @@
     <parent link="chasis"/>
     <child link="gps_link"/>
-    <origin xyz="0.0 0.0 0.3" rpy="0 0 0"/>
+    <origin xyz="0.0 0.0 0.0" rpy="0 0 0"/>
   </joint>
   <gazebo reference="gps_link">
@@ -411,12 +375,6 @@
         <velocity_sensing>true</velocity_sensing>
       </gps>
-      <plugin name="gps_plugin" filename="libgazebo_ros_gps.so">
-        <ros>
-          <namespace>/rosbot</namespace>
-          <remapping>~/gps/fix:=/gps/fix</remapping>
-          <update_rate>1.0</update_rate>
-        </ros>
-      </plugin>
     </sensor>
   </gazebo>
+  <xacro:include filename="gazebo.xacro"/>
 </robot>

Commit message: actualizacion 6

File: src/rosbot/urdf/include.xacro (robot description, xacro)
@@ -14,27 +14,95 @@
         <color rgba="0 0 0 1"/>
     </material>
-    <!-- Especificar colores de gazebo -->
+    <!-- Especificaciones de gazebo -->
     <gazebo reference="chasis">
         <material>Gazebo/Blue</material>
     </gazebo>
+    <gazebo reference="master">
+        <material>Gazebo/Blue</material>
+    </gazebo>
+    <gazebo reference="lidar_link">
+        <material>Gazebo/Black</material>
+    </gazebo>
     <gazebo reference="right_wheel">
         <material>Gazebo/White</material>
-        <mu1>0.2</mu1>
-        <mu2>0.2</mu2>
     </gazebo>
     <gazebo reference="left_wheel">
         <material>Gazebo/White</material>
-        <mu1>0.2</mu1>
-        <mu2>0.2</mu2>
     </gazebo>
     <gazebo reference="right_wheel_front">
         <material>Gazebo/White</material>
-        <mu1>0.2</mu1>
-        <mu2>0.2</mu2>
     </gazebo>
     <gazebo reference="left_wheel_front">
         <material>Gazebo/White</material>
-        <mu1>0.2</mu1>
-        <mu2>0.2</mu2>
+    </gazebo>
+    <gazebo reference="camera_link">
+        <sensor name="depth_camera" type="depth">
+            <visualize>true</visualize>
+            <update_rate>30.0</update_rate>
+            <camera name="camera">
+                <horizontal_fov>1.047198</horizontal_fov>
+                <image>
+                    <width>640</width>
+                    <height>480</height>
+                    <format>R8G8B8</format>
+                </image>
+                <clip>
+                    <near>0.05</near>
+                    <far>3</far>
+                </clip>
+            </camera>
+            <plugin name="depth_camera_controller" filename="libgazebo_ros_camera.so">
+                <baseline>0.2</baseline>
+                <alwaysOn>true</alwaysOn>
+                <updateRate>0.0</updateRate>
+                <frameName>camera_depth_frame</frameName>
+                <pointCloudCutoff>0.5</pointCloudCutoff>
+                <pointCloudCutoffMax>3.0</pointCloudCutoffMax>
+                <distortionK1>0</distortionK1>
+                <distortionK2>0</distortionK2>
+                <distortionK3>0</distortionK3>
+                <distortionT1>0</distortionT1>
+                <distortionT2>0</distortionT2>
+                <CxPrime>0</CxPrime>
+                <Cx>0</Cx>
+                <Cy>0</Cy>
+                <focalLength>0</focalLength>
+                <hackBaseline>0</hackBaseline>
+            </plugin>
+        </sensor>
+    </gazebo>
+    <gazebo reference="lidar_link">
+        <sensor name="lidar" type="ray">
+            <always_on>true</always_on>
+            <visualize>true</visualize>
+            <update_rate>5</update_rate>
+            <ray>
+                <scan>
+                    <horizontal>
+                        <samples>120</samples>
+                        <resolution>1.000000</resolution>
+                        <min_angle>-3.14159</min_angle>
+                        <max_angle>3.14159</max_angle>
+                    </horizontal>
+                </scan>
+                <range>
+                    <min>0.3</min>
+                    <max>15.0</max>
+                    <resolution>0.015</resolution>
+                </range>
+                <noise>
+                    <type>gaussian</type>
+                    <mean>0.0</mean>
+                    <stddev>0.01</stddev>
+                </noise>
+            </ray>
+            <plugin name="scan" filename="libgazebo_ros_ray_sensor.so">
+                <ros>
+                    <remapping>~/out:=scan</remapping>
+                </ros>
+                <output_type>sensor_msgs/LaserScan</output_type>
+                <frame_name>lidar_link</frame_name>
+            </plugin>
+        </sensor>
     </gazebo>
     <!-- Macro para calcular la inercia de un chasis rectangular -->

File: src/rosbot/urdf/rosbot.urdf.xacro (robot description, xacro)
@@ -80,9 +80,23 @@
   </joint>
   <link name="master">
+    <visual>
+      <geometry>
+        <box size="0.001 0.001 0.001"/>
+      </geometry>
+      <material name="blue"/>
+    </visual>
+    <collision>
+      <geometry>
+        <box size="0.001 0.001 0.001"/>
+      </geometry>
+    </collision>
+    <xacro:inertial_box mass="0.181" x="0.1" y="0.1" z="0.2">
+      <origin xyz="0 0 0" rpy="0 0 0"/>
+    </xacro:inertial_box>
   </link>
   <joint name="master_joint" type="revolute">
     <parent link="chasis"/>
     <child link="master"/>
-    <origin xyz="0 0 0" rpy= "1.57 0 0"/>
+    <origin xyz="0.24 0 0" rpy= "1.57 0 0"/>
     <axis xyz="0 1 0"/>
     <limit effort="100" velocity="1" lower="-0.78" upper="0.78"/>
@@ -207,42 +221,6 @@
     <child link="camera_depth_frame"/>
   </joint>
-  <gazebo reference="camera_link">
-    <sensor name="depth_camera" type="depth">
-      <visualize>true</visualize>
-      <update_rate>30.0</update_rate>
-      <camera name="camera">
-        <horizontal_fov>1.047198</horizontal_fov>
-        <image>
-          <width>640</width>
-          <height>480</height>
-          <format>R8G8B8</format>
-        </image>
-        <clip>
-          <near>0.05</near>
-          <far>3</far>
-        </clip>
-      </camera>
-      <plugin name="depth_camera_controller" filename="libgazebo_ros_camera.so">
-        <baseline>0.2</baseline>
-        <alwaysOn>true</alwaysOn>
-        <updateRate>0.0</updateRate>
-        <frameName>camera_depth_frame</frameName>
-        <pointCloudCutoff>0.5</pointCloudCutoff>
-        <pointCloudCutoffMax>3.0</pointCloudCutoffMax>
-        <distortionK1>0</distortionK1>
-        <distortionK2>0</distortionK2>
-        <distortionK3>0</distortionK3>
-        <distortionT1>0</distortionT1>
-        <distortionT2>0</distortionT2>
-        <CxPrime>0</CxPrime>
-        <Cx>0</Cx>
-        <Cy>0</Cy>
-        <focalLength>0</focalLength>
-        <hackBaseline>0</hackBaseline>
-      </plugin>
-    </sensor>
-  </gazebo>
   <!--lidar-->
-   <link name="lidar_link">
+  <link name="lidar_link">
     <inertial>
       <origin xyz="0 0 0" rpy="0 0 0"/>
@@ -268,113 +246,4 @@
     <origin xyz=" 0.2 0 0.15" rpy="0 0 0"/>
   </joint>
-  <gazebo reference="lidar_link">
-    <sensor name="lidar" type="ray">
-      <always_on>true</always_on>
-      <visualize>true</visualize>
-      <update_rate>5</update_rate>
-      <ray>
-        <scan>
-          <horizontal>
-            <samples>120</samples>
-            <resolution>1.000000</resolution>
-            <min_angle>-3.14159</min_angle>
-            <max_angle>3.14159</max_angle>
-          </horizontal>
-        </scan>
-        <range>
-          <min>0.3</min>
-          <max>15.0</max>
-          <resolution>0.015</resolution>
-        </range>
-        <noise>
-          <type>gaussian</type>
-          <mean>0.0</mean>
-          <stddev>0.01</stddev>
-        </noise>
-      </ray>
-      <plugin name="scan" filename="libgazebo_ros_ray_sensor.so">
-        <ros>
-          <remapping>~/out:=scan</remapping>
-        </ros>
-        <output_type>sensor_msgs/LaserScan</output_type>
-        <frame_name>lidar_link</frame_name>
-      </plugin>
-    </sensor>
-  </gazebo>
-  <gazebo reference="lidar_link">
-    <mu1>0.01</mu1>
-    <mu2>0.01</mu2>
-    <material>Gazebo/Black</material>
-  </gazebo>
-  <!-- IMU -->
-  <link name="imu_link">
-    <inertial>
-      <mass value="0.01"/>
-      <inertia ixx="0.001" ixy="0" ixz="0" iyy="0.001" iyz="0" izz="0.001"/>
-    </inertial>
-    <visual>
-      <geometry>
-        <box size="0.03 0.03 0.01"/>
-      </geometry>
-      <origin xyz="0 0 0" rpy="0 0 0"/>
-      <material name="grey"/>
-    </visual>
-  </link>
-  <joint name="imu_joint" type="fixed">
-    <parent link="chasis"/>
-    <child link="imu_link"/>
-    <origin xyz="0.0 0.0 0.0" rpy="0 0 0"/>
-  </joint>
-  <gazebo reference="imu_link">
-    <sensor type="imu" name="imu_sensor">
-      <update_rate>50.0</update_rate>
-      <imu>
-        <angular_velocity>
-          <x>true</x>
-          <y>true</y>
-          <z>true</z>
-        </angular_velocity>
-        <linear_acceleration>
-          <x>true</x>
-          <y>true</y>
-          <z>true</z>
-        </linear_acceleration>
-        <orientation>
-          <x>true</x>
-          <y>true</y>
-          <z>true</z>
-        </orientation>
-      </imu>
-    </sensor>
-  </gazebo>
-  <!-- GPS -->
-  <link name="gps_link">
-    <inertial>
-      <origin xyz="0 0 0" rpy="0 0 0"/>
-      <mass value="0.01"/>
-      <inertia ixx="0.001" ixy="0" ixz="0" iyy="0.001" iyz="0" izz="0.001"/>
-    </inertial>
-    <visual>
-      <geometry>
-        <box size="0.05 0.05 0.01"/>
-      </geometry>
-      <origin xyz="0 0 0" rpy="0 0 0"/>
-      <material name="grey"/>
-    </visual>
-  </link>
-  <joint name="gps_joint" type="fixed">
-    <parent link="chasis"/>
-    <child link="gps_link"/>
-    <origin xyz="0.0 0.0 0.0" rpy="0 0 0"/>
-  </joint>
-  <gazebo reference="gps_link">
-    <sensor type="gps" name="gps_sensor">
-      <update_rate>1.0</update_rate>
-      <gps>
-        <position_sensing>true</position_sensing>
-        <velocity_sensing>true</velocity_sensing>
-      </gps>
-    </sensor>
-  </gazebo>
   <xacro:include filename="gazebo.xacro"/>
 </robot>
