Commit message: actualizacion 7

File: src/rosbot/urdf/include.xacro (robot description, xacro)
@@ -13,4 +13,7 @@
     <material name="grey">
         <color rgba="0 0 0 1"/>
+    </material>
+    <material name="black">
+        <color rgba="0.0 0.0 0.0 0.0"/>
     </material>
     <!-- Especificaciones de gazebo -->
@@ -37,57 +40,45 @@
     </gazebo>
     <gazebo reference="camera_link">
-        <sensor name="depth_camera" type="depth">
+        <material>Gazebo/Red</material>
+        <sensor name="camera" type="depth">
+            <pose> 0 0 0 0 0 0 </pose>
             <visualize>true</visualize>
-            <update_rate>30.0</update_rate>
-            <camera name="camera">
-                <horizontal_fov>1.047198</horizontal_fov>
+            <update_rate>10</update_rate>
+            <camera>
+                <horizontal_fov>1.089</horizontal_fov>
                 <image>
+                    <format>B8G8R8</format>
                     <width>640</width>
                     <height>480</height>
-                    <format>R8G8B8</format>
                 </image>
                 <clip>
                     <near>0.05</near>
-                    <far>3</far>
+                    <far>8.0</far>
                 </clip>
             </camera>
-            <plugin name="depth_camera_controller" filename="libgazebo_ros_camera.so">
-                <baseline>0.2</baseline>
-                <alwaysOn>true</alwaysOn>
-                <updateRate>0.0</updateRate>
-                <frameName>camera_depth_frame</frameName>
-                <pointCloudCutoff>0.5</pointCloudCutoff>
-                <pointCloudCutoffMax>3.0</pointCloudCutoffMax>
-                <distortionK1>0</distortionK1>
-                <distortionK2>0</distortionK2>
-                <distortionK3>0</distortionK3>
-                <distortionT1>0</distortionT1>
-                <distortionT2>0</distortionT2>
-                <CxPrime>0</CxPrime>
-                <Cx>0</Cx>
-                <Cy>0</Cy>
-                <focalLength>0</focalLength>
-                <hackBaseline>0</hackBaseline>
+            <plugin name="camera_controller" filename="libgazebo_ros_camera.so">
+                <frame_name>camera_link_optical</frame_name>
+                <min_depth>0.1</min_depth>
+                <max_depth>100.0</max_depth>
             </plugin>
         </sensor>
     </gazebo>
-    <gazebo reference="lidar_link">
-        <sensor name="lidar" type="ray">
-            <always_on>true</always_on>
+    <gazebo reference="laser_frame">
+        <material>Gazebo/Black</material>
+        <sensor name="laser" type="ray">
+            <pose> 0 0 0 0 0 0 </pose>
             <visualize>true</visualize>
-            <update_rate>5</update_rate>
+            <update_rate>10</update_rate>
             <ray>
                 <scan>
                     <horizontal>
                         <samples>120</samples>
-                        <resolution>1.000000</resolution>
-                        <min_angle>-3.14159</min_angle>
-                        <max_angle>3.14159</max_angle>
+                        <min_angle>-3.14</min_angle>
+                        <max_angle>3.14</max_angle>
                     </horizontal>
                 </scan>
                 <range>
                     <min>0.3</min>
-                    <max>15.0</max>
-                    <resolution>0.015</resolution>
+                    <max>12</max>
                 </range>
                 <noise>
@@ -97,10 +88,10 @@
                 </noise>
             </ray>
-            <plugin name="scan" filename="libgazebo_ros_ray_sensor.so">
+            <plugin name="laser_controller" filename="libgazebo_ros_ray_sensor.so">
                 <ros>
-                    <remapping>~/out:=scan</remapping>
+                    <argument>~/out:=scan</argument>
                 </ros>
                 <output_type>sensor_msgs/LaserScan</output_type>
-                <frame_name>lidar_link</frame_name>
+                <frame_name>laser_frame</frame_name>
             </plugin>
         </sensor>

File: src/rosbot/urdf/rosbot.urdf.xacro (robot description, xacro)
@@ -53,4 +53,5 @@
     <origin xyz="-0.27 -0.295 -0.07" rpy="1.57 0 0"/>
     <axis xyz="0 0 1"/>
+    <dynamics damping="0.0" friction="0.1"/>
   </joint>
  <!--Left -->
@@ -78,4 +79,5 @@
     <origin xyz="-0.27 0.295 -0.07" rpy="1.57 0 0"/>
     <axis xyz="0 0 1"/>
+    <dynamics damping="0.0" friction="0.1"/>
   </joint>
   <link name="master">
@@ -100,4 +102,5 @@
     <origin xyz="0.24 0 0" rpy= "1.57 0 0"/>
     <axis xyz="0 1 0"/>
+    <dynamics damping="0.0" friction="0.1"/>
     <limit effort="100" velocity="1" lower="-0.78" upper="0.78"/>
   </joint>
@@ -137,4 +140,5 @@
     <origin xyz="0.27 -0.295 -0.07" rpy="1.57 0 0"/>
     <axis xyz="0 1 0"/>
+    <dynamics damping="0.0" friction="0.1"/>
     <limit effort="100" velocity="1" lower="-0.78" upper="0.78"/>
     <mimic joint="master_joint" multiplier="1.0" offset="0"/>
@@ -145,4 +149,5 @@
     <origin xyz="0.0 0 0" rpy="0 0 0"/>
     <axis xyz="0 0 1"/>
+    <dynamics damping="0.0" friction="0.1"/>
     <limit effort="100" velocity="1"/>
   </joint>
@@ -190,7 +195,13 @@
     <origin xyz="0.0 0 0" rpy="0 0 0"/>
     <axis xyz="0 0 1"/>
+    <dynamics damping="0.0" friction="0.1"/>
     <limit effort="100" velocity="1"/>
   </joint>
   <!--camara-->
+  <joint name="camera_joint" type="fixed">
+    <parent link="chasis"/>
+    <child link="camera_link"/>
+    <origin xyz="0.276 0 0.181" rpy="0 0.18 0"/>
+  </joint>
   <link name="camera_link">
     <visual>
@@ -200,50 +211,43 @@
       </geometry>
     </visual>
-    <collision>
-      <origin xyz="0 0 0" rpy="0 -0.156 0"/>
-      <geometry>
-        <box size="0.04 0.17 0.03"/>
-      </geometry>
-    </collision>
     <xacro:inertial_box mass="0.181" x="0.04" y="0.17" z="0.03">
       <origin xyz="0 0 0" rpy="0 0 0"/>
     </xacro:inertial_box>
   </link>
-  <joint name="camera_joint" type="fixed">
-    <parent link="chasis"/>
-    <child link="camera_link"/>
-    <origin xyz=" 0.30 0 0.1" rpy="0 -0.156 0"/>
-  </joint>
-  <link name="camera_depth_frame"/>
-  <joint name="camera_depth_joint" type="fixed">
-    <origin xyz="0 0 0" rpy="0 0 0"/>
+  <joint name="camera_optical_joint" type="fixed">
     <parent link="camera_link"/>
-    <child link="camera_depth_frame"/>
-  </joint>
+    <child link="camera_link_optical"/>
+    <origin xyz="0 0 0" rpy="1.57 0 1.57"/>
+  </joint>
+  <link name="camera_link_optical"></link>
   <!--lidar-->
-  <link name="lidar_link">
-    <inertial>
-      <origin xyz="0 0 0" rpy="0 0 0"/>
-      <mass value="0.125"/>
-      <inertia ixx="0.001"  ixy="0"  ixz="0" iyy="0.001" iyz="0" izz="0.001" />
-    </inertial>
-    <collision>
-      <origin xyz="0 0 0" rpy="0 0 0"/>
-      <geometry>
-         <cylinder radius="0.05" length="0.05"/>
-      </geometry>
-    </collision>
-    <visual>
-      <origin xyz="0 0 0" rpy="0 0 0"/>
-      <geometry>
-         <cylinder radius="0.05" length="0.09"/>
-      </geometry>
-    </visual>
-  </link>
-  <joint name="lidar_joint" type="fixed">
-    <parent link="chasis"/>
-    <child link="lidar_link"/>
-    <origin xyz=" 0.2 0 0.15" rpy="0 0 0"/>
-  </joint>
+  <joint name="laser_joint" type="fixed">
+    <parent link="chasis"/>
+    <child link="laser_frame"/>
+    <origin xyz="0.2 0 0.15" rpy="0 0 0"/>
+  </joint>
+  <link name="laser_frame">
+    <visual>
+      <geometry>
+        <cylinder radius="0.05" length="0.04"/>
+      </geometry>
+      <material name="black"/>
+    </visual>
+    <visual>
+      <origin xyz="0 0 -0.05"/>
+      <geometry>
+        <cylinder radius="0.01" length="0.1"/>
+      </geometry>
+      <material name="black"/>
+    </visual>
+    <collision>
+      <geometry>
+        <cylinder radius="0.05" length="0.04"/>
+      </geometry>
+    </collision>
+    <xacro:inertial_cylinder mass="0.1" length="0.04" radius="0.05">
+        <origin xyz="0 0 0" rpy="0 0 0"/>
+    </xacro:inertial_cylinder>
+  </link>
   <xacro:include filename="gazebo.xacro"/>
 </robot>
