Commit message: actualizacion 9

File: src/rosbot/urdf/gazebo.xacro (robot description, xacro)
@@ -33,6 +33,6 @@
         <joint name="master_joint">
             <command_interface name="position">
-                <param name="min">-1.5708</param> <!-- -90 degrees -->
-                <param name="max">1.5708</param>  <!-- +90 degrees -->
+                <param name="min">-0.349</param> <!-- -20 degrees -->
+                <param name="max">0.349</param>  <!-- +20 degrees -->
             </command_interface>
             <state_interface name="position"/>

File: src/rosbot/urdf/include.xacro (robot description, xacro)
@@ -20,4 +20,5 @@
     <gazebo reference="chasis">
         <material>Gazebo/Blue</material>
+        <gravity>1</gravity>
     </gazebo>
     <gazebo reference="master">
@@ -28,14 +29,26 @@
     </gazebo>
     <gazebo reference="right_wheel">
+        <mu1 value="0.001"/>
+        <mu2 value="0.01"/>
         <material>Gazebo/White</material>
+        <gravity>1</gravity>
     </gazebo>
     <gazebo reference="left_wheel">
+        <mu1 value="0.001"/>
+        <mu2 value="0.01"/>
         <material>Gazebo/White</material>
+        <gravity>1</gravity>
     </gazebo>
     <gazebo reference="right_wheel_front">
+        <mu1 value="0.001"/>
+        <mu2 value="0.01"/>
         <material>Gazebo/White</material>
+        <gravity>1</gravity>
     </gazebo>
     <gazebo reference="left_wheel_front">
+        <mu1 value="0.001"/>
+        <mu2 value="0.01"/>
         <material>Gazebo/White</material>
+        <gravity>1</gravity>
     </gazebo>
     <gazebo reference="camera_link">
@@ -74,6 +87,6 @@
                     <horizontal>
                         <samples>120</samples>
-                        <min_angle>-3.14</min_angle>
-                        <max_angle>3.14</max_angle>
+                        <min_angle>-3.1</min_angle>
+                        <max_angle>3.1</max_angle>
                     </horizontal>
                 </scan>

File: src/rosbot/urdf/rosbot.urdf.xacro (robot description, xacro)
@@ -25,6 +25,6 @@
     <inertial>
       <origin xyz="-0.381 0.2 -0.075" rpy = "1.57 0 0"/>
-      <mass value="30"/>
-      <inertia  ixx="456250.0" ixy="0" ixz="0" iyy="1844000.0" iyz="0" izz="1500250.0" />
+      <mass value="35"/>
+      <inertia  ixx="532291666.6666666" ixy="0" ixz="0" iyy="2151333333.333333" iyz="0" izz="1750291666.6666665" />
     </inertial>
   </link>
@@ -51,5 +51,5 @@
     <parent link="chasis"/>
     <child link="right_wheel"/>
-    <origin xyz="-0.27 -0.295 -0.07" rpy="1.57 0 0"/>
+    <origin xyz="-0.27 -0.295 -0.06" rpy="1.57 0 0"/>
     <axis xyz="0 0 1"/>
     <dynamics damping="0.0" friction="0.1"/>
@@ -77,5 +77,5 @@
     <parent link="chasis"/>
     <child link="left_wheel"/>
-    <origin xyz="-0.27 0.295 -0.07" rpy="1.57 0 0"/>
+    <origin xyz="-0.27 0.295 -0.06" rpy="1.57 0 0"/>
     <axis xyz="0 0 1"/>
     <dynamics damping="0.0" friction="0.1"/>
@@ -93,5 +93,5 @@
       </geometry>
     </collision>
-    <xacro:inertial_box mass="0.181" x="0.1" y="0.1" z="0.2">
+    <xacro:inertial_box mass="0.001" x="0.01" y="00.1" z="0.01">
       <origin xyz="0 0 0" rpy="0 0 0"/>
     </xacro:inertial_box>
@@ -102,5 +102,4 @@
     <origin xyz="0.24 0 0" rpy= "1.57 0 0"/>
     <axis xyz="0 1 0"/>
-    <dynamics damping="0.0" friction="0.1"/>
     <limit effort="100" velocity="1" lower="-0.78" upper="0.78"/>
   </joint>
@@ -108,9 +107,13 @@
     <visual>
       <geometry>
-         <cylinder length="0.001" radius="0.04"/>
-      </geometry>
-      <origin xyz="0 0 0"/>
-      <material name="white"/>
-    </visual>
+        <cylinder length="0.001" radius="0.04"/>
+      </geometry>
+      <material name="white"/>
+    </visual>
+    <collision>
+      <geometry>
+        <cylinder length="0.001" radius="0.04"/>
+      </geometry>
+    </collision>
     <xacro:inertial_cylinder mass="1.0" length="0.001" radius="0.04">
       <origin xyz="0 0 0" rpy="0 0 0"/>
@@ -120,11 +123,9 @@
     <visual>
       <geometry>
-         <cylinder length="0.08" radius="0.12"/>
-      </geometry>
-      <origin xyz="0 0 0"/>
-      <material name="white"/>
-    </visual>
-    <collision>
-      <origin xyz="0 0 0"/>
+        <cylinder length="0.08" radius="0.12"/>
+      </geometry>
+      <material name="white"/>
+    </visual>
+    <collision>
       <geometry>
         <cylinder length="0.08" radius="0.12"/>
@@ -138,5 +139,5 @@
     <parent link="chasis"/>
     <child link="right_wheel_front_assembly"/>
-    <origin xyz="0.27 -0.295 -0.07" rpy="1.57 0 0"/>
+    <origin xyz="0.27 -0.295 -0.06" rpy="1.57 0 0"/>
     <axis xyz="0 1 0"/>
     <dynamics damping="0.0" friction="0.1"/>
@@ -149,9 +150,10 @@
     <origin xyz="0.0 0 0" rpy="0 0 0"/>
     <axis xyz="0 0 1"/>
-    <dynamics damping="0.0" friction="0.1"/>
+    <dynamics damping="0.0" friction="1"/>
     <limit effort="100" velocity="1"/>
   </joint>
+ <!--  -->
   <link name="left_wheel_front_assembly">
-      <visual>
+    <visual>
       <geometry>
          <cylinder length="0.001" radius="0.04"/>
@@ -160,4 +162,10 @@
       <material name="white"/>
     </visual>
+    <collision>
+      <origin xyz="0 0 0"/>
+      <geometry>
+        <cylinder length="0.001" radius="0.04"/>
+      </geometry>
+    </collision>
     <xacro:inertial_cylinder mass="1.0" length="0.001" radius="0.04">
       <origin xyz="0 0 0" rpy="0 0 0"/>
@@ -167,5 +175,5 @@
     <visual>
       <geometry>
-         <cylinder length="0.08" radius="0.12"/>
+        <cylinder length="0.08" radius="0.12"/>
       </geometry>
       <origin xyz="0 0 0"/>
@@ -185,15 +193,15 @@
     <parent link="chasis"/>
     <child link="left_wheel_front_assembly"/>
-    <origin xyz="0.27 0.295 -0.07" rpy="1.57 0 0"/>
+    <origin xyz="0.27 0.295 -0.06" rpy="1.57 0 0"/>
     <axis xyz="0 1 0"/>
     <limit effort="100" velocity="1" lower="-0.78" upper="0.78"/>
     <mimic joint="master_joint" multiplier="1.0" offset="0"/>
   </joint>
-    <joint name="left_wheel_joint" type="continuous">
+  <joint name="left_wheel_joint" type="continuous">
     <parent link="left_wheel_front_assembly"/>
     <child link="left_wheel_front"/>
     <origin xyz="0.0 0 0" rpy="0 0 0"/>
     <axis xyz="0 0 1"/>
-    <dynamics damping="0.0" friction="0.1"/>
+    <dynamics damping="0.0" friction="1"/>
     <limit effort="100" velocity="1"/>
   </joint>
@@ -211,6 +219,12 @@
       </geometry>
     </visual>
+    <collision>
+      <origin xyz="0 0 0" rpy="0 -0.156 0"/>
+      <geometry>
+        <box size="0.04 0.17 0.03"/>
+      </geometry>
+    </collision>
     <xacro:inertial_box mass="0.181" x="0.04" y="0.17" z="0.03">
-      <origin xyz="0 0 0" rpy="0 0 0"/>
+      <origin xyz="0 0 0" rpy="0 -0.156 0"/>
     </xacro:inertial_box>
   </link>
@@ -218,5 +232,5 @@
     <parent link="camera_link"/>
     <child link="camera_link_optical"/>
-    <origin xyz="0 0 0" rpy="1.57 0 1.57"/>
+    <origin xyz="0 0 0" rpy="-1.57 0 -1.57"/>
   </joint>
   <link name="camera_link_optical"></link>
@@ -234,11 +248,4 @@
       <material name="black"/>
     </visual>
-    <visual>
-      <origin xyz="0 0 -0.05"/>
-      <geometry>
-        <cylinder radius="0.01" length="0.1"/>
-      </geometry>
-      <material name="black"/>
-    </visual>
     <collision>
       <geometry>
@@ -246,5 +253,5 @@
       </geometry>
     </collision>
-    <xacro:inertial_cylinder mass="0.1" length="0.04" radius="0.05">
+    <xacro:inertial_cylinder mass="0.3" length="0.04" radius="0.05">
         <origin xyz="0 0 0" rpy="0 0 0"/>
     </xacro:inertial_cylinder>

Commit message: actualizacion 10 / Cambio de controlador

File: src/rosbot/urdf/gazebo.xacro (robot description, xacro)
@@ -30,16 +30,16 @@
             <param name="initial_velocity">0.0</param>
         </joint>
-        <!-- Define the steering wheel joint (for direction control) -->
+        <!-- Define the steering wheel joint (for direction control)
         <joint name="master_joint">
             <command_interface name="position">
-                <param name="min">-0.349</param> <!-- -20 degrees -->
-                <param name="max">0.349</param>  <!-- +20 degrees -->
+                <param name="min">-0.349</param>
+                <param name="max">0.349</param>
             </command_interface>
             <state_interface name="position"/>
             <param name="initial_position">0.0</param>
-        </joint>
+        </joint>-->
         <!-- Define the steering wheel joint (for direction control) -->
         <joint name="joint_left_wheel_front">
-            <param name="mimic">master_joint</param>
+            <!--<param name="mimic">master_joint</param>-->
             <param name="multiplier">1</param>
             <command_interface name="position"/>
@@ -48,5 +48,5 @@
             <!-- Define the steering wheel joint (for direction control) -->
         <joint name="joint_right_wheel_front">
-            <param name="mimic">master_joint</param>
+            <!--<param name="mimic">master_joint</param>-->
             <param name="multiplier">1</param>
             <command_interface name="position"/>

File: src/rosbot/urdf/include.xacro (robot description, xacro)
@@ -29,24 +29,36 @@
     </gazebo>
     <gazebo reference="right_wheel">
-        <mu1 value="0.001"/>
-        <mu2 value="0.01"/>
+        <mu1 value="1.0"/>
+        <mu2 value="1.0"/>
+        <kp  value="10000000.0" />
+        <kd  value="1.0" />
+        <fdir1 value="1 0 0"/>
         <material>Gazebo/White</material>
         <gravity>1</gravity>
     </gazebo>
     <gazebo reference="left_wheel">
-        <mu1 value="0.001"/>
-        <mu2 value="0.01"/>
+        <mu1 value="1.0"/>
+        <mu2 value="1.0"/>
+        <kp  value="10000000.0" />
+        <kd  value="1.0" />
+        <fdir1 value="1 0 0"/>
         <material>Gazebo/White</material>
         <gravity>1</gravity>
     </gazebo>
     <gazebo reference="right_wheel_front">
-        <mu1 value="0.001"/>
-        <mu2 value="0.01"/>
+        <mu1 value="1.0"/>
+        <mu2 value="1.0"/>
+        <kp  value="10000000.0" />
+        <kd  value="1.0" />
+        <fdir1 value="0 0 1"/>
         <material>Gazebo/White</material>
         <gravity>1</gravity>
     </gazebo>
     <gazebo reference="left_wheel_front">
-        <mu1 value="0.001"/>
-        <mu2 value="0.01"/>
+        <mu1 value="1.0"/>
+        <mu2 value="1.0"/>
+        <kp  value="10000000.0" />
+        <kd  value="1.0" />
+        <fdir1 value="0 0 1"/>
         <material>Gazebo/White</material>
         <gravity>1</gravity>

File: src/rosbot/urdf/rosbot.urdf.xacro (robot description, xacro)
@@ -143,5 +143,5 @@
     <dynamics damping="0.0" friction="0.1"/>
     <limit effort="100" velocity="1" lower="-0.78" upper="0.78"/>
-    <mimic joint="master_joint" multiplier="1.0" offset="0"/>
+    <!--<mimic joint="master_joint" multiplier="1.0" offset="0"/>-->
   </joint>
   <joint name="right_wheel_joint" type="continuous">
@@ -196,5 +196,5 @@
     <axis xyz="0 1 0"/>
     <limit effort="100" velocity="1" lower="-0.78" upper="0.78"/>
-    <mimic joint="master_joint" multiplier="1.0" offset="0"/>
+    <!--<mimic joint="master_joint" multiplier="1.0" offset="0"/>-->
   </joint>
   <joint name="left_wheel_joint" type="continuous">
